File: Mono-Test-Pcb.kicad_pcb (KiCad board)
At the start: 2 copper layers, 11 parts, among them J1 AudioJack4_Ground, U1 ESP32-C6-DevKitM-1

Commit message: isolamento dos sinais adc
Parts:
- moved J1 87.6 mm to (236.1, 59.8), turned to 180 degrees
- moved C1 76.5 mm to (235.1, 42.4), turned to 0 degrees
- moved REF** 68.4 mm to (229.9, 88.3)
- moved R2 67.1 mm to (230.9, 44.2)
- moved D2 51.9 mm to (219.8, 53.2)
- moved R1 37.0 mm to (215.6, 40.5), turned to 0 degrees
- moved D1 36.0 mm to (215.9, 49.0), turned to 0 degrees
- moved REF** 35.7 mm to (180.6, 42.6)
- moved OUT1 33.8 mm to (179.2, 57.2), turned to -90 degrees
- moved REF** 23.1 mm to (180.6, 88.3)
Connections:
- U1 pad 29: unconnected-(U1-GPIO2-Pad29) -> Net-(D1-A)
- U1 pad 5: Net-(D1-A) -> Net-(OUT1-Pin_2)
- U1 pad 9: Net-(OUT1-Pin_2) -> unconnected-(U1-GPIO1-Pad9)
Routing:
- net Net-(D1-A): track 56.4 -> 27.7 mm
- net Net-(D1-K): track 74.4 -> 53.7 mm
- net Net-(OUT1-Pin_2): track 30.6 -> 10.1 mm
- net Net-(C1-Pad1): track 33.4 -> 26.8 mm
