File: Mono-Test-Pcb.kicad_sch (KiCad schematic)
At the start: 8 parts, among them J1 AudioJack4_Ground, U1 ESP32-C6-DevKitM-1

Commit message: isolamento dos sinais adc
Connections:
- net at D1.2 (A), D2.1 (K), J1.T: now also U1.29 (GPIO2); no longer U1.5 (GPIO5)
- net at OUT1.2 (Pin_2): now also U1.5 (GPIO5); no longer U1.9 (GPIO1)
Other:
- moved on the sheet: C1, D1, D2, J1, R1, R2
